File: SteinerParkerVCF/YuSynth-SteinerParkerVCF.kicad_sch (KiCad schematic)
At the start: 53 parts, among them J1 EURO_PWR_2x5, J11 Conn_01x05_Male, J8 Conn_01x08_Female, Q1 BC547, Q2 BC547, U1 TL074

Commit message: modif pcb
Parts:
- removed R19: 3.9K, Resistor_THT:R_Axial_DIN0207_L6.3mm_D2.5mm_P5.08mm_Vertical, symbol Device:R
- added RV9: 100K, Potentiometer_THT:Potentiometer_Bourns_3266Y_Vertical, symbol Device:R_Potentiometer_Trim
Connections:
- net RESONANCE CW-MainB: now also RV9.2, RV9.3
- net at C16.1, R16.2, U1.8: now also RV9.1
Changed lines of the file:
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@@
   (junction (at 125.73 58.42) (diameter 0) (color 0 0 0 0)
   )
+  (junction (at 227.33 35.56) (diameter 0) (color 0 0 0 0)
+  )
   (junction (at 146.05 71.12) (diameter 0) (color 0 0 0 0)
   )
@@
     (stroke (width 0) (type default) (color 0 0 0 0))
   )
+  (wire (pts (xy 222.25 39.37) (xy 227.33 39.37))
+    (stroke (width 0) (type default) (color 0 0 0 0))
+  )
   (wire (pts (xy 257.81 20.32) (xy 261.62 20.32))
     (stroke (width 0) (type default) (color 0 0 0 0))
@@
     (stroke (width 0) (type default) (color 0 0 0 0))
   )
+  (wire (pts (xy 226.06 35.56) (xy 227.33 35.56))
+    (stroke (width 0) (type default) (color 0 0 0 0))
+  )
   (wire (pts (xy 240.03 132.08) (xy 240.03 140.97))
     (stroke (width 0) (type default) (color 0 0 0 0))
@@
     (stroke (width 0) (type default) (color 0 0 0 0))
   )
-  (wire (pts (xy 222.25 39.37) (xy 222.25 49.53))
-    (stroke (width 0) (type default) (color 0 0 0 0))
-  )
   (wire (pts (xy 99.06 83.82) (xy 99.06 86.36))
     (stroke (width 0) (type default) (color 0 0 0 0))
@@
     (stroke (width 0) (type default) (color 0 0 0 0))
   )
+  (wire (pts (xy 227.33 39.37) (xy 227.33 35.56))
+    (stroke (width 0) (type default) (color 0 0 0 0))
+  )
   (wire (pts (xy 207.01 31.75) (xy 189.23 31.75))
     (stroke (width 0) (type default) (color 0 0 0 0))
@@
     (stroke (width 0) (type default) (color 0 0 0 0))
   )
+  (wire (pts (xy 227.33 35.56) (xy 229.87 35.56))
+    (stroke (width 0) (type default) (color 0 0 0 0))
+  )
   (wire (pts (xy 100.33 29.21) (xy 115.57 29.21))
+    (stroke (width 0) (type default) (color 0 0 0 0))
+  )
+  (wire (pts (xy 229.87 35.56) (xy 229.87 49.53))
     (stroke (width 0) (type default) (color 0 0 0 0))
   )
@@
     )
   )
-  (global_label "RESONANCE CW-MainB" (shape input) (at 222.25 49.53 0) (fields_autoplaced)
+  (global_label "RESONANCE CW-MainB" (shape input) (at 229.87 49.53 0) (fields_autoplaced)
     (effects (font (size 1.27 1.27)) (justify left))
-    (property "Références Inter-Feuilles" "${INTERSHEET_REFS}" (id 0) (at 246.6764 49.4506 0)
+    (property "Références Inter-Feuilles" "${INTERSHEET_REFS}" (id 0) (at 254.2964 49.4506 0)
       (effects (font (size 1.27 1.27)) (justify left) hide)
     )
@@
   (symbol (lib_id "Amplifier_Operational:TL074") (at 214.63 29.21 0) (mirror x) (unit 3)
     (in_bom yes) (on_board yes)
-    (property "Reference" "U1" (id 0) (at 214.63 36.83 0))
-    (property "Value" "TL074" (id 1) (at 214.63 39.37 0))
+    (property "Reference" "U1" (id 0) (at 210.82 35.56 0))
+    (property "Value" "TL074" (id 1) (at 210.82 38.1 0))
     (property "Footprint" "Package_DIP:DIP-14_W7.62mm_LongPads" (id 2) (at 213.36 31.75 0)
       (effects (font (size 1.27 1.27)) hide)
@@
     (pin "2")
   )
-  (symbol (lib_id "Device:R") (at 222.25 35.56 180) (unit 1)
-    (in_bom yes) (on_board yes) (fields_autoplaced)
-    (property "Reference" "R19" (id 0) (at 224.79 34.2899 0)
-      (effects (font (size 1.27 1.27)) (justify right))
-    )
-    (property "Value" "3.9K" (id 1) (at 224.79 36.8299 0)
-      (effects (font (size 1.27 1.27)) (justify right))
-    )
-    (property "Footprint" "Resistor_THT:R_Axial_DIN0207_L6.3mm_D2.5mm_P5.08mm_Vertical" (id 2) (at 224.028 35.56 90)
-      (effects (font (size 1.27 1.27)) hide)
-    )
-    (property "Datasheet" "~" (id 3) (at 222.25 35.56 0)
-      (effects (font (size 1.27 1.27)) hide)
-    )
-    (pin "1")
-    (pin "2")
-  )
   (symbol (lib_id "eurorack:EURO_PWR_2x5") (at 252.73 146.05 0) (unit 1)
     (in_bom yes) (on_board yes) (fields_autoplaced)
@@
     (pin "2")
   )
+  (symbol (lib_id "Device:R_Potentiometer_Trim") (at 222.25 35.56 0) (unit 1)
+    (in_bom yes) (on_board yes) (fields_autoplaced)
+    (property "Reference" "RV9" (id 0) (at 219.71 34.2899 0)
+      (effects (font (size 1.27 1.27)) (justify right))
+    )
+    (property "Value" "100K" (id 1) (at 219.71 36.8299 0)
+      (effects (font (size 1.27 1.27)) (justify right))
+    )
+    (property "Footprint" "Potentiometer_THT:Potentiometer_Bourns_3266Y_Vertical" (id 2) (at 222.25 35.56 0)
+      (effects (font (size 1.27 1.27)) hide)
+    )
+    (property "Datasheet" "~" (id 3) (at 222.25 35.56 0)
+      (effects (font (size 1.27 1.27)) hide)
+    )
+    (pin "1")
+    (pin "2")
+    (pin "3")
+  )
   (symbol (lib_id "Device:R") (at 220.98 152.4 90) (unit 1)
     (in_bom yes) (on_board yes) (fields_autoplaced)
@@
     )
     (path "/97577e2e-bf29-4e34-97e9-b9b8211ece7c/638f17fd-ea4f-4ea8-8988-c2e4480ab3a8"
-      (reference "111") (unit 1) (value "SR1712F-0204-20F0A-N9-N-027") (footprint "Button_Switch_THT:SR1712F020420F0AN9N027")
+      (reference "1111") (unit 1) (value "SR1712F-0204-20F0A-N9-N-027") (footprint "Button_Switch_THT:SR1712F020420F0AN9N027")
     )
     (path "/b22d337f-231a-421f-800f-d240448c494a"
@@
       (reference "R18") (unit 1) (value "10") (footprint "Resistor_THT:R_Axial_DIN0207_L6.3mm_D2.5mm_P5.08mm_Vertical")
     )
-    (path "/cc17f343-fee9-4181-8279-a4e397f6de77"
-      (reference "R19") (unit 1) (value "3.9K") (footprint "Resistor_THT:R_Axial_DIN0207_L6.3mm_D2.5mm_P5.08mm_Vertical")
-    )
     (path "/83b568fc-9b53-45ab-8157-4cffc1c901c8"
       (reference "R20") (unit 1) (value "10K") (footprint "Resistor_THT:R_Axial_DIN0207_L6.3mm_D2.5mm_P5.08mm_Vertical")
@@
       (reference "RV8") (unit 1) (value "RESONANCE 50K REV-AUDIO") (footprint "Potentiometer_THT:Potentiometer_Alpha_RD901F-40-00D_Single_Vertical")
     )
+    (path "/ee8dbbf9-9eb8-4f7d-8d54-44069ddb15aa"
+      (reference "RV9") (unit 1) (value "100K") (footprint "Potentiometer_THT:Potentiometer_Bourns_3266Y_Vertical")
+    )
     (path "/504f5041-82af-49ea-9980-4e5790bd6830"
